Commit message: feat: minor fix & auto pipeline

File: objects/toilet/102703_evogen/mobility_revised.urdf (robot description, URDF)
Before this commit: robot partnet_ed38aee3026bee7a3321831d2245cf06, 6 links, 5 joints
Joints:
- joint joint_2: limit lower=-0.0 upper=1.7453292519943295 -> lower=-0.0 upper=1.75
- joint joint_3: limit lower=-0.0 upper=1.6929693744344996 -> lower=-0.0 upper=1.70

File: objects/toilet/102703_vlm1shot/mobility_revised.urdf (robot description, URDF)
Before this commit: robot partnet_ed38aee3026bee7a3321831d2245cf06, 6 links, 5 joints
Joints:
- joint joint_2: limit lower=0.0 upper=1.7453 -> lower=0.0 upper=1.75
- joint joint_3: limit lower=0.0 upper=1.693 -> lower=0.0 upper=1.70
