Commit message: version saved after submission

File: objects/cabinet/19179_evogen/mobility_revised.urdf (robot description, URDF)
Before this commit: robot partnet_1314c9a583812b9fc0eea8e38540939d, 4 links, 3 joints
Links:
- link link_0: mass 8.4 -> 2.0; geometry collision mesh filename=textured_objs/original_10.obj scale=0.250000 0.250000 0.250000; collision mesh filename=textured_objs/original_11.obj scale=0.250000 0.250000 0.250000
- link link_1: mass 8.4 -> 2.0; geometry collision mesh filename=textured_objs/original_13.obj scale=0.250000 0.250000 0.250000; collision mesh filename=textured_objs/original_14.obj scale=0.250000 0.250000 0.250000
- link link_2: mass 70.0 -> 8.0; geometry collision mesh filename=textured_objs/original_1.obj scale=0.250000 0.250000 0.250000; collision mesh filename=textured_objs/original_4.obj scale=0.250000 0.250000 0.250000
Joints:
- joint joint_0: limit lower=0 upper=1 -> lower=-0.02 upper=0.25
- joint joint_1: limit lower=0 upper=1 -> lower=-0.02 upper=0.25

File: objects/cabinet/19179_ivw/mobility_revised.urdf (robot description, URDF)
Before this commit: robot partnet_1314c9a583812b9fc0eea8e38540939d, 4 links, 3 joints
Links:
- link link_0: mass 3.962338291248703 -> 2.2570329670329667; geometry collision mesh filename=textured_objs/original_10.obj scale=0.420137 0.420137 0.420137; collision mesh filename=textured_objs/original_11.obj scale=0.420137 0.420137 0.420137
- link link_1: mass 4.056256983240224 -> 2.271868131868132; geometry collision mesh filename=textured_objs/original_13.obj scale=0.420137 0.420137 0.420137; collision mesh filename=textured_objs/original_14.obj scale=0.420137 0.420137 0.420137
- link link_2: mass 23.40531608763222 -> 11.598034206017614; geometry collision mesh filename=textured_objs/original_1.obj scale=0.420137 0.420137 0.420137; collision mesh filename=textured_objs/original_4.obj scale=0.420137 0.420137 0.420137
Joints:
- joint joint_0: limit lower=0.0 upper=0.9999999999999917 -> lower=0.0 upper=0.2770825426944971
- joint joint_1: limit lower=0.0 upper=0.9999999999999917 -> lower=0.0 upper=0.2770825426944971

File: objects/cabinet/19179_vlm1shot/mobility_revised.urdf (robot description, URDF)
Before this commit: robot partnet_1314c9a583812b9fc0eea8e38540939d, 4 links, 3 joints
Links:
- link link_0: mass 2.5 -> 1.0; geometry collision mesh filename=textured_objs/original_10.obj scale=0.454500 0.454500 0.454500; collision mesh filename=textured_objs/original_11.obj scale=0.454500 0.454500 0.454500
- link link_1: mass 2.5 -> 1.0; geometry collision mesh filename=textured_objs/original_13.obj scale=0.454500 0.454500 0.454500; collision mesh filename=textured_objs/original_14.obj scale=0.454500 0.454500 0.454500
- link link_2: mass 20.0 -> 13.0; geometry collision mesh filename=textured_objs/original_1.obj scale=0.454500 0.454500 0.454500; collision mesh filename=textured_objs/original_4.obj scale=0.454500 0.454500 0.454500
Joints:
- joint joint_0: limit lower=0.0 upper=0.5 -> lower=0.0 upper=0.22
- joint joint_1: limit lower=0.0 upper=0.5 -> lower=0.0 upper=0.22

File: objects/trashcan/102181_ivw/mobility_revised.urdf (robot description, URDF)
Before this commit: robot partnet_8766d229-05d2-4609-902f-66ce6dc510fa, 4 links, 3 joints
Joints:
- joint joint_1: limit lower=-3.309366666666607e-16 upper=2.189450877272629e-14 -> lower=0.0 upper=3.1541590242041524
